File: pcb/dicecalc/dicecalc.sch (KiCad schematic (older format))
At the start: 125 parts, among them J1 Conn_01x19_Female, J2 Conn_01x19_Female, J3 Conn_01x19_Female, J4 Conn_01x19_Female, J5 Conn_01x10_Male, SW1 SW_Push, SW10 SW_Push, SW11 SW_Push, SW12 SW_Push, SW13 SW_Push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

Commit message: Note pins that need to move
Other:
- note added: "CLRs: Move to other place"
Changed lines of the file:
@@
 Text Notes 3300 8200 0    50   ~ 0
 PD2 Located here
+Text Notes 5200 9850 0    50   ~ 0
+CLRs: Move to other place
 $EndSCHEMATC
