File: pcb/entropy/entropy.sch (KiCad schematic (older format))
At the start: 23 parts, among them J1 Conn_01x04_Male, U1 TPS61041DBV, U2 LM358, U3 TLV3201

Commit message: Add random test
Other:
- note added: "Connect to other diode terminal"
- note added: "Connect to other diode terminal\n"
Changed lines of the file:
@@
 	1    0    0    -1
 $EndComp
+Text Notes 8150 2500 0    100  ~ 0
+Connect to other diode terminal\n
+Text Notes 8150 4050 0    100  ~ 0
+Connect to other diode terminal
 $EndSCHEMATC
